File: hardware/schematic_esp8266_basic.kicad_sch (KiCad schematic)
At the start: 18 parts, among them J1 AUDIO_JACK_2.5MMSPECIAL_POGO_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, U1 SI4735-D60-GU, U2 ESP8266, Y1 CRYSTALPTH-2X6

Commit message: new file:   hardware/fp-info-cache 	new file:   hardware/schematic_esp8266_basic-backups/schematic_esp8266_basic-2025-01-23_105310.zip 	new file:   hardware/schematic_esp8266_basic.kicad_pcb 	modified:   hardware/schematic_esp8266_basic.kicad_prl 	modified:   hardware/schematic_esp8266_basic.kicad_pro 	modified:   hardware/schematic_esp8266_basic.kicad_sch
Parts:
- L1: renamed from #L1; symbol schematic_esp8266_basic-eagle-import:L -> Device:L
